Commit message: second commit

File: cb_description/urdf/cb.urdf.xacro (robot description, xacro)
@@ -3,13 +3,11 @@
   <!-- arguments -->
   <xacro:arg name="robot_namespace" default="/"/>
-  <xacro:arg name="kinect1_enabled" default="true"/>
-  <xacro:arg name="kinect2_enabled" default="false"/>
-  <xacro:arg name="realsense1_enabled" default="false"/>
+  <xacro:arg name="realsense1_enabled" default="true"/>
   <xacro:arg name="realsense2_enabled" default="true"/>
+  <xacro:arg name="realsense3_enabled" default="true"/>
   <xacro:arg name="ur_enabled" default="true"/>
   <xacro:arg name="gripper_enabled" default="true"/>
   <!-- components -->
   <xacro:include filename="$(find cb_description)/urdf/components/inspector_bot.urdf.xacro" />
-  <xacro:include filename="$(find cb_description)/urdf/accessories/kinect_tilted_camera.urdf.xacro"/>
   <xacro:include filename="$(find ur_description)/urdf/ur5.urdf.xacro" />
   <xacro:include filename="$(find robotiq_2f_85_gripper_visualization)/urdf/robotiq_arg2f_85_model_macro.xacro" />
@@ -52,53 +50,50 @@
   </xacro:if>
   <!-- ********************* -->
-  <!--         kinect        -->
-  <!-- ********************* -->
-  <xacro:if value="$(arg kinect1_enabled)">
-    <xacro:arg name="kinect1_base_xyz" default="${base_x_size/2 + 0.041} 0 ${base_center_height + base_z_size/2 - 0.071}"/>
-    <xacro:arg name="kinect1_base_rpy" default="0 0 0"/>
-    <xacro:arg name="kinect1_tilt_angle" default="0"/>
-    <xacro:kinect_tilted_camera prefix="kinect1" robot_namespace="$(arg robot_namespace)"
-      base_xyz="$(arg kinect1_base_xyz)" base_rpy="$(arg kinect1_base_rpy)" tilt_angle="$(arg kinect1_tilt_angle)"/>
-  </xacro:if>
-  <xacro:if value="$(arg kinect2_enabled)">
-    <xacro:property name="kinect2_height" value="0.40"/>
-    <xacro:arg name="kinect2_base_xyz" default="${-base_x_size/2 - profile_size/2 + 0.03} ${-base_y_size/2 + profile_size*1.5} ${base_center_height + base_z_size/2 + kinect2_height}"/>
-    <!-- <xacro:arg name="kinect2_base_rpy" default="0 0 -0.785"/> -->
-    <xacro:arg name="kinect2_base_rpy" default="0 0 -0.795"/>
-    <!-- <xacro:arg name="kinect2_tilt_angle" default="-0.471"/> -->
-    <xacro:arg name="kinect2_tilt_angle" default="-0.42"/>
-    <xacro:kinect_tilted_camera prefix="kinect2" robot_namespace="$(arg robot_namespace)"
-      base_xyz="$(arg kinect2_base_xyz)" base_rpy="$(arg kinect2_base_rpy)" tilt_angle="$(arg kinect2_tilt_angle)"/>
-  </xacro:if>
-  <!-- ********************* -->
   <!--       realsense       -->
   <!-- ********************* -->
   <xacro:if value="$(arg realsense1_enabled)">
-    <link name="realsense1_mount_link" />
-    <joint name="realsense1_profile_fixed_joint" type="fixed">
-      <parent link="camera_profile"/>
-      <child link="realsense1_mount_link"/>
-      <origin xyz="0 0 ${profile_height1/2}" rpy="0 0 ${-M_PI/4}"/>
-    </joint>
     <link name="realsense1_base_link" />
     <joint name="realsense1_mount_fixed_joint" type="fixed">
-      <parent link="realsense1_mount_link"/>
+      <parent link="ee_link"/>
       <child link="realsense1_base_link"/>
+      <origin xyz="-0.02 0.065 0.0" rpy="${-M_PI/2} 0 0"/>
+    </joint>
+    <xacro:sensor_d415 parent="realsense1_base_link" name="realsense1">
+      <origin xyz="0 0 0" rpy="0 0 0"/>
+    </xacro:sensor_d415>
+  </xacro:if>
+  <xacro:if value="$(arg realsense2_enabled)">
+    <link name="realsense2_mount_link" />
+    <joint name="realsense2_profile_fixed_joint" type="fixed">
+      <parent link="camera_profile_left"/>
+      <child link="realsense2_mount_link"/>
+      <origin xyz="0 0 ${profile_left_height/2}" rpy="0 0 ${M_PI/4}"/>
+    </joint>
+    <link name="realsense2_base_link" />
+    <joint name="realsense2_mount_fixed_joint" type="fixed">
+      <parent link="realsense2_mount_link"/>
+      <child link="realsense2_base_link"/>
       <origin xyz="0.035 0 0.025" rpy="0 ${M_PI/6} 0"/>
     </joint>
-    <xacro:sensor_d435 parent="realsense1_base_link" name="realsense1">
+    <xacro:sensor_d435 parent="realsense2_base_link" name="realsense2">
       <origin xyz="0.010 0 -0.0125" rpy="0 0 0"/>
     </xacro:sensor_d435>
   </xacro:if>
-  <xacro:if value="$(arg realsense2_enabled)">
-    <link name="realsense2_base_link" />
-    <joint name="realsense2_mount_fixed_joint" type="fixed">
-      <parent link="ee_link"/>
-      <child link="realsense2_base_link"/>
-      <origin xyz="-0.02 0.065 0.0" rpy="${-M_PI/2} 0 0"/>
+  <xacro:if value="$(arg realsense3_enabled)">
+    <link name="realsense3_mount_link" />
+    <joint name="realsense3_profile_fixed_joint" type="fixed">
+      <parent link="camera_profile_right"/>
+      <child link="realsense3_mount_link"/>
+      <origin xyz="0 0 ${profile_right_height/2}" rpy="0 0 ${-M_PI/4}"/>
     </joint>
-    <xacro:sensor_d415 parent="realsense2_base_link" name="realsense2">
-      <origin xyz="0 0 0" rpy="0 0 0"/>
-    </xacro:sensor_d415>
+    <link name="realsense3_base_link" />
+    <joint name="realsense3_mount_fixed_joint" type="fixed">
+      <parent link="realsense3_mount_link"/>
+      <child link="realsense3_base_link"/>
+      <origin xyz="0.035 0 0.025" rpy="0 ${M_PI/6} 0"/>
+    </joint>
+    <xacro:sensor_d435 parent="realsense3_base_link" name="realsense3">
+      <origin xyz="0.010 0 -0.0125" rpy="0 0 0"/>
+    </xacro:sensor_d435>
   </xacro:if>
 </robot>

File: cb_description/urdf/components/gripper_for_int_marker.urdf.xacro (robot description, xacro)
@@ -5,5 +5,5 @@
     <origin rpy="0.0 0 0" xyz="0 0 0"/>
     <geometry>
-      <mesh filename="package://mm_description/meshes/gripper/robotiq_2f85_opened_combined_axis_mated.STL"/>
+      <mesh filename="package://cb_description/meshes/gripper/robotiq_2f85_opened_combined_axis_mated.STL"/>
     </geometry>
   </visual>

File: cb_description/urdf/components/inspector_bot.urdf.xacro (robot description, xacro)
@@ -2,5 +2,5 @@
 <robot name="inspector_bot" xmlns:xacro="http://ros.org/wiki/xacro">
   <!-- Materials -->
-  <xacro:include filename="$(find mm_description)/urdf/common_properties.xacro" />
+  <xacro:include filename="$(find cb_description)/urdf/common_properties.xacro" />
   <!-- Base Size -->
   <xacro:property name="base_x_size" value="0.76" />
@@ -9,5 +9,6 @@
   <!-- Profile Size -->
   <xacro:property name="profile_size" value="0.04" />
-  <xacro:property name="profile_height1" value="${0.415+0.077}"/> <!-- camera -->
+  <xacro:property name="profile_left_height" value="0.2"/> <!-- camera -->
+  <xacro:property name="profile_right_height" value="0.7"/> <!-- camera -->
   <!-- Origin -->
   <xacro:property name="origin_x" value="0.025" />
@@ -119,14 +120,14 @@
     <origin xyz="${-wheelbase/2} ${-track/2} ${wheel_vertical_offset}" rpy="0 0 0" />
   </xacro:inspector_bot_wheel>
-  <!-- profile for side facing camera -->
-  <!-- <joint name="camera_profile_fixed_joint" type="fixed">
+  <!-- profile for side facing camera : left, right-->
+  <joint name="camera_profile_left_fixed_joint" type="fixed">
     <parent link="bare_base_link"/>
-    <child link="camera_profile"/>
-    <origin xyz="${-base_x_size/2 - profile_size/2} ${-base_y_size/2 + profile_size*1.5} ${base_center_height + base_z_size/2 + profile_height1/2}" rpy="0 0 0"/>
+    <child link="camera_profile_left"/>
+    <origin xyz="${-base_x_size/2 + profile_size/2} ${base_y_size/2 - profile_size/2} ${base_center_height + base_z_size/2 + profile_left_height/2}" rpy="0 0 0"/>
   </joint>
-  <link name="camera_profile">
+  <link name="camera_profile_left">
     <visual>
       <geometry>
-        <box size="${profile_size} ${profile_size} ${profile_height1}"/>
+        <box size="${profile_size} ${profile_size} ${profile_left_height}"/>
       </geometry>
       <material name="black"/>
@@ -134,11 +135,30 @@
     <collision>
       <geometry>
-        <box size="${profile_size} ${profile_size} ${profile_height1}"/>
+        <box size="${profile_size} ${profile_size} ${profile_left_height}"/>
       </geometry>
       <material name="black"/>
     </collision>
-  </link> -->
+  </link>
+  <joint name="camera_profile_right_fixed_joint" type="fixed">
+    <parent link="bare_base_link"/>
+    <child link="camera_profile_right"/>
+    <origin xyz="${-base_x_size/2 + profile_size/2} ${-base_y_size/2 + profile_size/2} ${base_center_height + base_z_size/2 + profile_right_height/2}" rpy="0 0 0"/>
+  </joint>
+  <link name="camera_profile_right">
+    <visual>
+      <geometry>
+        <box size="${profile_size} ${profile_size} ${profile_right_height}"/>
+      </geometry>
+      <material name="black"/>
+    </visual>
+    <collision>
+      <geometry>
+        <box size="${profile_size} ${profile_size} ${profile_right_height}"/>
+      </geometry>
+      <material name="black"/>
+    </collision>
+  </link>
   <!-- battery -->
-  <joint name="camera_profile_fixed_joint" type="fixed">
+  <joint name="battery_fixed_joint" type="fixed">
     <parent link="bare_base_link"/>
     <child link="battery_link"/>

Commit message: success from capture to scan execute

File: cb_description/urdf/cb.urdf.xacro (robot description, xacro)
@@ -5,5 +5,5 @@
   <xacro:arg name="realsense1_enabled" default="true"/>
   <xacro:arg name="realsense2_enabled" default="true"/>
-  <xacro:arg name="realsense3_enabled" default="true"/>
+  <xacro:arg name="realsense3_enabled" default="false"/>
   <xacro:arg name="ur_enabled" default="true"/>
   <xacro:arg name="gripper_enabled" default="true"/>
@@ -20,8 +20,18 @@
     <xacro:property name="ur5_z_location" value="${base_center_height + base_z_size/2}" />
     <xacro:property name="ur5_x_location" value="0.175" />
-    <joint name="ur_fixed_joint" type="fixed">
+    <link name="real_base_link"/>
+    <link name="real_ee_link"/>
+    <link name="tcp_gripper_open"/>
+    <link name="tcp_gripper_closed"/>
+    <link name="uv_light_center"/>
+    <joint name="ur_real_base_fixed_joint" type="fixed">
       <parent link="bare_base_link" />
+      <child link="real_base_link" />
+      <origin xyz="${ur5_x_location} 0.0 ${ur5_z_location}" rpy="0.0 0.0 ${M_PI/2}" />
+    </joint>
+    <joint name="ur_base_fixed_joint" type="fixed">
+      <parent link="real_base_link" />
       <child link="base_link" />
-      <origin xyz="${ur5_x_location} 0.0 ${ur5_z_location}" rpy="0.0 0.0 -${M_PI/2}" />
+      <origin xyz="0.0 0.0 0.0" rpy="0.0 0.0 -${M_PI}" />
     </joint>
     <joint name="ur_real_ee_fixed_joint" type="fixed">
@@ -30,5 +40,19 @@
       <origin xyz="0.0 0.0 0.0" rpy="-${M_PI/2} 0.0 -${M_PI/2}" />
     </joint>
-    <link name="real_ee_link"/>
+    <joint name="ur_tcp_fixed_joint" type="fixed">
+      <parent link="real_ee_link"/>
+      <child link="tcp_gripper_open"/>
+      <origin xyz="0 0 0.13" rpy="0 0 0"/>
+    </joint>
+    <joint name="ur_gripper_closed_fixed_joint" type="fixed">
+      <parent link="tcp_gripper_open"/>
+      <child link="tcp_gripper_closed"/>
+      <origin xyz="0 0 0.01" rpy="0 0 0"/>
+    </joint>
+    <joint name="ur_light_center_fixed_joint" type="fixed">
+      <parent link="tcp_gripper_closed"/>
+      <child link="uv_light_center"/>
+      <origin xyz="-0.155 0 0" rpy="0 0 0"/>
+    </joint>
     <xacro:ur5_robot prefix="" joint_limited="false"/>
     <!-- gripper -->
@@ -39,5 +63,4 @@
         <origin xyz="0 0 0" rpy="0 0 0"/>
       </joint>
-      <!-- actual end-effector -->
       <joint name="ur_ee_fixed_joint" type="fixed">
         <parent link="tool0"/>

File: cb_description/urdf/components/inspector_bot.urdf.xacro (robot description, xacro)
@@ -25,5 +25,6 @@
   <xacro:property name="battery_x_size" value="${0.18+0.02}"/>
   <xacro:property name="battery_y_size" value="${0.36+0.02}"/>
-  <xacro:property name="battery_z_size" value="${0.28+0.02}"/>
+  <!-- <xacro:property name="battery_z_size" value="${0.28+0.02}"/> -->
+  <xacro:property name="battery_z_size" value="${0.28-0.02}"/>
   <xacro:property name="M_PI" value="3.14159"/>
   <!-- Inspector_bot wheel macro -->
@@ -140,10 +141,10 @@
     </collision>
   </link>
-  <joint name="camera_profile_right_fixed_joint" type="fixed">
+  <!-- <joint name="camera_profile_right_fixed_joint" type="fixed">
     <parent link="bare_base_link"/>
     <child link="camera_profile_right"/>
     <origin xyz="${-base_x_size/2 + profile_size/2} ${-base_y_size/2 + profile_size/2} ${base_center_height + base_z_size/2 + profile_right_height/2}" rpy="0 0 0"/>
-  </joint>
-  <link name="camera_profile_right">
+  </joint> -->
+  <!-- <link name="camera_profile_right">
     <visual>
       <geometry>
@@ -158,5 +159,5 @@
       <material name="black"/>
     </collision>
-  </link>
+  </link> -->
   <!-- battery -->
   <joint name="battery_fixed_joint" type="fixed">
