Commit message: demo version update

File: cb_description/urdf/accessories/kinect_tilted_camera.urdf.xacro (robot description, xacro)
@@ -57,5 +57,5 @@
         <origin xyz="-0.021 -0.0325 -0.019" rpy="0 0 ${M_PI/2}"/>
         <geometry>
-          <mesh filename="package://mm_description/meshes/accessories/kinect.dae" />
+          <mesh filename="package://cb_description/meshes/accessories/kinect.dae" />
         </geometry>
       </visual>

File: cb_description/urdf/cb.urdf.xacro (robot description, xacro)
@@ -6,4 +6,5 @@
   <xacro:arg name="realsense2_enabled" default="true"/>
   <xacro:arg name="realsense3_enabled" default="false"/>
+  <xacro:arg name="kinect1_enabled" default="true"/>
   <xacro:arg name="ur_enabled" default="true"/>
   <xacro:arg name="gripper_enabled" default="true"/>
@@ -14,4 +15,5 @@
   <xacro:include filename="$(find realsense2_description)/urdf/_d415.urdf.xacro" />
   <xacro:include filename="$(find realsense2_description)/urdf/_d435.urdf.xacro" />
+  <xacro:include filename="$(find cb_description)/urdf/accessories/kinect_tilted_camera.urdf.xacro"/>
   <!-- ********************* -->
   <!--          ur5          -->
@@ -120,3 +122,13 @@
     </xacro:sensor_d435>
   </xacro:if>
+  <!-- ********************* -->
+  <!--         kinect        -->
+  <!-- ********************* -->
+  <xacro:if value="$(arg kinect1_enabled)">
+    <xacro:arg name="kinect1_base_xyz" default="${base_x_size/2 + 0.041} 0 ${base_center_height + base_z_size/2 - 0.071}"/>
+    <xacro:arg name="kinect1_base_rpy" default="0 0 0"/>
+    <xacro:arg name="kinect1_tilt_angle" default="0"/>
+    <xacro:kinect_tilted_camera prefix="kinect1" robot_namespace="$(arg robot_namespace)"
+      base_xyz="$(arg kinect1_base_xyz)" base_rpy="$(arg kinect1_base_rpy)" tilt_angle="$(arg kinect1_tilt_angle)"/>
+  </xacro:if>
 </robot>
